File: pcb/airpcb_smd/airpcb_smd.kicad_pcb (KiCad board)
At the start: 2 copper layers, 49 x 65 mm, 21 parts, among them J1 SPI, J2 DHT, J4 AB, J7 PWR, J8 WS2812, Q1 PN2222A, Q2 PN2222A, U1 PC817, U2 PC817, U3 NodeMCU_ESP-12E

Commit message: placed in one side
Parts:
- J1, J2, J4, J7, J8, U1, U2, U3: moved to B.Cu
- moved J8 40.4 mm to (157.5, 90.2), turned to 0 degrees
- moved J1 40.4 mm to (157.5, 106.2), turned to 180 degrees
- moved J2 40.4 mm to (157.5, 94.1), turned to 180 degrees
- moved J7 39.5 mm to (117.9, 87.9)
- moved U3 29.4 mm to (122.6, 115.9), turned to 0 degrees
- moved R7 25.9 mm to (146.6, 110.2)
- moved D2 15.8 mm to (146.6, 103.6)
- moved U2 15.2 mm to (129.7, 90.4)
- moved R4 15.1 mm to (127.5, 85.9), turned to 180 degrees
- moved R1 14.9 mm to (145.5, 86.1), turned to 0 degrees
- moved U1 14.0 mm to (144.3, 98.0)
- moved R3 11.2 mm to (142.0, 108.7)
- moved Q2 10.7 mm to (135.4, 112.8)
- moved D3 8.81 mm to (130.3, 116.1)
- moved D1 7.52 mm to (131.8, 104.1), turned to -90 degrees
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Routing:
- net GND: track 129.4 -> 52.8 mm
- net 3V3: track 113.0 -> 48.0 mm
- net 5V: track 59.4 -> 5.70 mm
- net A: track 43.8 -> 7.24 mm
- net B: track 32.1 -> 0.00 mm, vias 2 -> 0
- net Net-(D3-Pad1): track 27.1 -> 0.00 mm
- net D4: track 21.0 -> 0.00 mm
- net D3: track 16.0 -> 3.83 mm
- net Net-(D1-Pad1): track 15.1 -> 3.67 mm
- net Net-(D3-Pad2): track 7.70 -> 0.00 mm
- net SCL: track 6.98 -> 0.00 mm
- net SDA: track 6.98 -> 0.00 mm
- net Net-(Q2-Pad2): track 4.90 -> 0.00 mm
- net Net-(Q1-Pad2): track 5.04 -> 9.23 mm
- net Net-(D2-Pad2): track 2.78 -> 5.46 mm
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- removed copper zone on B.Cu, net 3V3
- removed copper zone on F.Cu, net 3V3
Other:
- board text removed: "3V"
- board text removed: "GND"
