File: pcb/kicad/airpcb_smd.kicad_sch (KiCad schematic)
At the start: 30 parts, among them J1 I2C, J11 PSU, J2 DHT, J3 DC, J4 AB, J7 PWR, J8 WS2812, J9 5V3V, Q1 PN2222A, Q2 PN2222A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

Commit message: pcb done
Parts:
- J4: footprint Connector_PinSocket_2.54mm:PinSocket_1x02_P2.54mm_Vertical -> TerminalBlock_Phoenix:TerminalBlock_Phoenix_MPT-0,5-2-2.54_1x02_P2.54mm_Horizontal
- Q1, Q2: footprint airpcb_smd:SOT-23_Reverse_Handsoldering -> Package_TO_SOT_SMD:TSOT-23_HandSoldering
Changed lines of the file:
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@@
       (effects (font (size 1.27 1.27)) (justify left))
     )
-    (property "Footprint" "airpcb_smd:SOT-23_Reverse_Handsoldering" (id 2) (at 93.98 126.365 0)
+    (property "Footprint" "Package_TO_SOT_SMD:TSOT-23_HandSoldering" (id 2) (at 93.98 126.365 0)
       (effects (font (size 1.27 1.27) italic) (justify left) hide)
     )
@@
       (effects (font (size 1.27 1.27)) (justify left))
     )
-    (property "Footprint" "airpcb_smd:SOT-23_Reverse_Handsoldering" (id 2) (at 57.15 118.745 0)
+    (property "Footprint" "Package_TO_SOT_SMD:TSOT-23_HandSoldering" (id 2) (at 57.15 118.745 0)
       (effects (font (size 1.27 1.27) italic) (justify left) hide)
     )
@@
       (effects (font (size 1.27 1.27)) (justify left))
     )
-    (property "Footprint" "Connector_PinSocket_2.54mm:PinSocket_1x02_P2.54mm_Vertical" (id 2) (at 149.733 42.037 0)
+    (property "Footprint" "TerminalBlock_Phoenix:TerminalBlock_Phoenix_MPT-0,5-2-2.54_1x02_P2.54mm_Horizontal" (id 2) (at 149.733 42.037 0)
       (effects (font (size 1.27 1.27)) hide)
     )
@@
     )
     (path "/00000000-0000-0000-0000-00005f5e144a"
-      (reference "J4") (unit 1) (value "AB") (footprint "Connector_PinSocket_2.54mm:PinSocket_1x02_P2.54mm_Vertical")
+      (reference "J4") (unit 1) (value "AB") (footprint "TerminalBlock_Phoenix:TerminalBlock_Phoenix_MPT-0,5-2-2.54_1x02_P2.54mm_Horizontal")
     )
     (path "/00000000-0000-0000-0000-00005f6377e8"
@@
     )
     (path "/00000000-0000-0000-0000-00005f584bbb"
-      (reference "Q1") (unit 1) (value "PN2222A") (footprint "airpcb_smd:SOT-23_Reverse_Handsoldering")
+      (reference "Q1") (unit 1) (value "PN2222A") (footprint "Package_TO_SOT_SMD:TSOT-23_HandSoldering")
     )
     (path "/00000000-0000-0000-0000-00005f571ed4"
-      (reference "Q2") (unit 1) (value "PN2222A") (footprint "airpcb_smd:SOT-23_Reverse_Handsoldering")
+      (reference "Q2") (unit 1) (value "PN2222A") (footprint "Package_TO_SOT_SMD:TSOT-23_HandSoldering")
     )
     (path "/00000000-0000-0000-0000-00005f5701ae"
